File: Controller_Mixer/pcb/controller_mixer_pcb/controller_mixer_pcb.kicad_pcb (KiCad board)
At the start: 2 copper layers, 26 parts, among them J1 Conn_01x08_Male, J10 Conn_01x08_Male, J15 Conn_01x05_Male, J16 Conn_01x05_Male, J17 Conn_01x04_Male, J18 Conn_01x04_Male, J19 Conn_01x08_Male, J2 Conn_01x08_Male, J20 Conn_01x08_Male, J3 Conn_01x08_Male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

Commit message: 1st Controller_Mixer pcb fertig
Parts:
- removed J17, J18, VU-LEDs1: Conn_01x04_Male, Connector_PinHeader_2.54mm:PinHeader_1x04_P2.54mm_Vertical
- added J5: Conn_01x05_Male, Connector_PinHeader_2.54mm:PinHeader_1x05_P2.54mm_Vertical, F.Cu at (190.5, 142.2)
- added J6: Conn_01x05_Male, Connector_PinHeader_2.54mm:PinHeader_1x05_P2.54mm_Vertical, F.Cu at (188.0, 129.5)
- added VUVs1: Conn_01x05_Male, Connector_PinHeader_2.54mm:PinHeader_1x05_P2.54mm_Vertical, F.Cu at (190.5, 138.4)
- VUs1: value Conn_01x04_Male -> Conn_01x05_Male; footprint Connector_PinHeader_2.54mm:PinHeader_1x04_P2.54mm_Vertical -> Connector_PinHeader_2.54mm:PinHeader_1x05_P2.54mm_Vertical
- moved MP1 231.5 mm to (264.2, 92.7), turned to 180 degrees
- moved MP2 206.4 mm to (238.8, 92.7), turned to 180 degrees
- moved J4 192.9 mm to (251.5, 62.2), turned to 90 degrees
- moved J2 189.8 mm to (251.5, 58.4), turned to 90 degrees
- moved J3 165.1 mm to (226.1, 62.2), turned to 90 degrees
- moved J1 161.4 mm to (226.1, 58.4), turned to 90 degrees
- moved U3 142.2 mm to (184.2, 109.2)
- moved MP3 136.6 mm to (213.4, 92.7), turned to 180 degrees
- moved J16 119.0 mm to (203.2, 129.5), turned to 270 degrees
- moved LEDs1 118.7 mm to (203.2, 125.7), turned to 270 degrees
- moved J15 117.4 mm to (219.7, 129.5), turned to 270 degrees
- moved BTNs1 117.0 mm to (219.7, 125.7), turned to 270 degrees
- moved R+|LED|T-1 115.5 mm to (161.3, 139.7), turned to 180 degrees
- moved MP4 111.7 mm to (188.0, 92.7), turned to 180 degrees
- moved T+|GND|R-1 110.8 mm to (165.1, 134.6)
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Connections:
- U3 pad 15: Net-(MP1-Pad16) -> Net-(U3-Pad15)
- U3 pad 46: Net-(U3-Pad46) -> Net-(MP1-Pad16)
Routing:
- net Net-(J1-Pad1): track 0.00 -> 482.6 mm
- net Net-(MP1-Pad9): track 0.00 -> 217.6 mm
- net Net-(MP1-Pad10): track 0.00 -> 215.2 mm
- net Net-(MP1-Pad11): track 0.00 -> 212.5 mm
- net Net-(MP1-Pad16): track 0.00 -> 130.8 mm
- net Net-(MP1-Pad3): track 0.00 -> 85.9 mm
- net Net-(MP2-Pad3): track 0.00 -> 61.7 mm
- net Net-(T+|GND|R-1-Pad3): track 0.00 -> 40.9 mm
- net Net-(J20-Pad8): track 0.00 -> 40.5 mm
- net Net-(R+|LED|T-1-Pad1): track 0.00 -> 39.7 mm
- net Net-(MP3-Pad3): track 0.00 -> 39.7 mm
- net Net-(J4-Pad8): track 0.00 -> 39.1 mm
- net Net-(J10-Pad8): track 0.00 -> 38.9 mm
- net Net-(J3-Pad8): track 0.00 -> 38.9 mm
- net Net-(J9-Pad8): track 0.00 -> 38.9 mm
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
Commit message: 1st Controller_Mixer pcb fertig
Parts:
- added R1: R_PHOTO, Resistor_THT:R_Axial_DIN0207_L6.3mm_D2.5mm_P5.08mm_Vertical, F.Cu at (196.8, 125.7)
- added R2: R_PHOTO, Resistor_THT:R_Axial_DIN0207_L6.3mm_D2.5mm_P5.08mm_Vertical, F.Cu at (200.7, 125.7)
- added R3: R_PHOTO, Resistor_THT:R_Axial_DIN0207_L6.3mm_D2.5mm_P5.08mm_Vertical, F.Cu at (204.5, 125.7)
- added R4: R_PHOTO, Resistor_THT:R_Axial_DIN0207_L6.3mm_D2.5mm_P5.08mm_Vertical, F.Cu at (208.3, 125.7)
- added R5: R_PHOTO, Resistor_THT:R_Axial_DIN0207_L6.3mm_D2.5mm_P5.08mm_Vertical, F.Cu at (193.0, 125.7)
- moved J16 13.3 mm to (207.0, 142.2)
- moved LEDs1 13.3 mm to (207.0, 138.4)
- moved J15 9.67 mm to (223.5, 120.7), turned to 0 degrees
- moved BTNs1 5.08 mm to (219.7, 120.7), turned to 0 degrees
Connections:
- U3 pad 16: Net-(LEDs1-Pad1) -> Net-(R5-Pad1)
- U3 pad 30: Net-(LEDs1-Pad2) -> Net-(R4-Pad1)
- U3 pad 31: Net-(LEDs1-Pad3) -> Net-(R3-Pad1)
- U3 pad 32: Net-(LEDs1-Pad4) -> Net-(R2-Pad1)
- U3 pad 33: Net-(LEDs1-Pad5) -> Net-(R1-Pad1)
Routing:
- net Net-(R4-Pad1): track 0.00 -> 27.3 mm
- net Net-(R3-Pad1): track 0.00 -> 27.2 mm
- net Net-(R2-Pad1): track 0.00 -> 26.2 mm
- net Net-(R1-Pad1): track 0.00 -> 25.7 mm
- net Net-(LEDs1-Pad5): track 25.1 -> 7.62 mm
- net Net-(LEDs1-Pad4): track 25.1 -> 8.15 mm
- net Net-(LEDs1-Pad3): track 25.1 -> 8.67 mm
- net Net-(J1-Pad1): track 482.6 -> 498.8 mm
- net Net-(LEDs1-Pad2): track 25.1 -> 9.20 mm
- net Net-(BTNs1-Pad5): track 26.8 -> 38.3 mm
- net Net-(R5-Pad1): track 0.00 -> 8.89 mm
- net Net-(BTNs1-Pad4): track 26.8 -> 33.2 mm
- net Net-(BTNs1-Pad1): track 26.8 -> 21.7 mm
- net Net-(BTNs1-Pad3): track 27.3 -> 29.7 mm
- net Net-(BTNs1-Pad2): track 26.8 -> 25.3 mm
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