File: Controller_Mixer/pcb/controller_mixer_pcb/controller_mixer_pcb.sch (KiCad schematic (older format))
At the start: 26 parts, among them J1 Conn_01x08_Male, J10 Conn_01x08_Male, J15 Conn_01x05_Male, J16 Conn_01x05_Male, J17 Conn_01x04_Male, J18 Conn_01x04_Male, J19 Conn_01x08_Male, J2 Conn_01x08_Male, J20 Conn_01x08_Male, J3 Conn_01x08_Male, J4 Conn_01x08_Male, J7 Conn_01x08_Male, J8 Conn_01x08_Male, J9 Conn_01x08_Male, U3 Teensy4.1

Commit message: 1st Controller_Mixer pcb fertig
Parts:
- removed J17, J18, VU-LEDs1, VUs1: Conn_01x04_Male, Connector_PinHeader_2.54mm:PinHeader_1x04_P2.54mm_Vertical, symbol Connector:Conn_01x04_Male
- added J5, J6, VUVs1, VUs1: Conn_01x05_Male, Connector_PinHeader_2.54mm:PinHeader_1x05_P2.54mm_Vertical, symbol Connector:Conn_01x05_Male
Connections:
- wire segments 211 -> 218
Changed lines of the file:
@@
 Wire Wire Line
 	7850 1550 7850 1650
-Connection ~ 7850 1650
 Wire Wire Line
 	4650 700  7150 700
@@
 Text GLabel 7950 2650 1    50   UnSpc ~ 0
 VU-CONNECTORS
-$Comp
-L Connector:Conn_01x04_Male J17
-U 1 1 5FB7A905
-P 7650 2250
-F 0 "J17" H 7758 2531 50  0000 C CNN
-F 1 "Conn_01x04_Male" H 7758 2440 50  0000 C CNN
-F 2 "Connector_PinHeader_2.54mm:PinHeader_1x04_P2.54mm_Vertical" H 7650 2250 50  0001 C CNN
-F 3 "~" H 7650 2250 50  0001 C CNN
-	1    7650 2250
-	1    0    0    -1
-$EndComp
-$Comp
-L Connector:Conn_01x04_Male VUs1
-U 1 1 5FB7E38C
-P 7600 2350
-F 0 "VUs1" H 7572 2232 50  0000 R CNN
-F 1 "Conn_01x04_Male" H 7572 2323 50  0000 R CNN
-F 2 "Connector_PinHeader_2.54mm:PinHeader_1x04_P2.54mm_Vertical" H 7600 2350 50  0001 C CNN
-F 3 "~" H 7600 2350 50  0001 C CNN
-	1    7600 2350
-	-1   0    0    1
-$EndComp
-Connection ~ 7850 2150
-Wire Wire Line
-	7850 2150 7850 2250
-Connection ~ 7850 2250
-Wire Wire Line
-	7850 2250 7850 2350
-Connection ~ 7850 2350
-Wire Wire Line
-	7850 2350 7850 2450
-Connection ~ 7850 2450
-$Comp
-L Connector:Conn_01x04_Male J18
-U 1 1 5FB8B727
-P 7650 3050
-F 0 "J18" H 7758 3331 50  0000 C CNN
-F 1 "Conn_01x04_Male" H 7758 3240 50  0000 C CNN
-F 2 "Connector_PinHeader_2.54mm:PinHeader_1x04_P2.54mm_Vertical" H 7650 3050 50  0001 C CNN
-F 3 "~" H 7650 3050 50  0001 C CNN
-	1    7650 3050
-	1    0    0    -1
-$EndComp
-Wire Wire Line
-	7850 2450 7850 2950
-Connection ~ 7850 2950
-Wire Wire Line
-	7850 2950 7850 3050
-Connection ~ 7850 3050
-Wire Wire Line
-	7850 3050 7850 3150
-Connection ~ 7850 3150
-Wire Wire Line
-	7850 3150 7850 3250
-Connection ~ 7850 3250
-Wire Wire Line
-	7850 3250 7850 3750
 Text GLabel 7950 3250 1    50   UnSpc ~ 0
 VU-LEDS
-Wire Wire Line
-	3750 3250 3750 3650
-Wire Wire Line
-	3750 3650 7150 3650
-Wire Wire Line
-	7150 3650 7150 2150
-Wire Wire Line
-	7150 2150 7400 2150
-Wire Wire Line
-	7400 2250 7100 2250
-Wire Wire Line
-	7100 2250 7100 3600
-Wire Wire Line
-	7100 3600 3850 3600
-Wire Wire Line
-	3850 3600 3850 3250
-Wire Wire Line
-	3950 3250 3950 3550
-Wire Wire Line
-	3950 3550 7050 3550
-Wire Wire Line
-	7050 3550 7050 2350
-Wire Wire Line
-	7050 2350 7400 2350
-Wire Wire Line
-	7400 2450 7000 2450
-Wire Wire Line
-	7000 2450 7000 3500
-Wire Wire Line
-	7000 3500 4050 3500
-Wire Wire Line
-	4050 3500 4050 3250
-Connection ~ 7400 3050
-Wire Wire Line
-	7400 3050 7400 3150
-Connection ~ 7400 3150
-Wire Wire Line
-	7400 3150 7400 3250
-Wire Wire Line
-	7400 3250 6950 3250
-Wire Wire Line
-	6950 3250 6950 3450
-Wire Wire Line
-	6950 3450 4150 3450
-Connection ~ 7400 3250
-Wire Wire Line
-	4150 4000 4300 4000
-Wire Wire Line
-	7400 3000 7400 3050
-Wire Wire Line
-	7400 2950 7400 3050
-Wire Wire Line
-	4150 3250 4150 3450
-Connection ~ 4150 3450
-Wire Wire Line
-	4150 3450 4150 4000
 Connection ~ 4300 4000
 $Comp
@@
 $EndComp
 Wire Wire Line
-	7850 1650 7850 2150
-Wire Wire Line
 	7850 1250 7850 1350
 Connection ~ 7850 1250
@@
 Wire Wire Line
 	7850 1350 7850 1450
-$Comp
-L Connector:Conn_01x04_Male VU-LEDs1
-U 1 1 5FB8B72D
+Wire Wire Line
+	2400 900  2950 900
+Wire Wire Line
+	2950 900  2950 1050
+$Comp
+L Connector:Conn_01x05_Male J5
+U 1 1 5FDC9B36
+P 7650 2350
+F 0 "J5" H 7758 2731 50  0000 C CNN
+F 1 "Conn_01x05_Male" H 7758 2640 50  0000 C CNN
+F 2 "Connector_PinHeader_2.54mm:PinHeader_1x05_P2.54mm_Vertical" H 7650 2350 50  0001 C CNN
+F 3 "~" H 7650 2350 50  0001 C CNN
+	1    7650 2350
+	1    0    0    -1
+$EndComp
+$Comp
+L Connector:Conn_01x05_Male VUs1
+U 1 1 5FDC9B3C
+P 7600 2350
+F 0 "VUs1" H 7572 2282 50  0000 R CNN
+F 1 "Conn_01x05_Male" H 7572 2373 50  0000 R CNN
+F 2 "Connector_PinHeader_2.54mm:PinHeader_1x05_P2.54mm_Vertical" H 7600 2350 50  0001 C CNN
+F 3 "~" H 7600 2350 50  0001 C CNN
+	1    7600 2350
+	-1   0    0    1
+$EndComp
+$Comp
+L Connector:Conn_01x05_Male J6
+U 1 1 5FE2A081
+P 7650 3150
+F 0 "J6" H 7758 3531 50  0000 C CNN
+F 1 "Conn_01x05_Male" H 7758 3440 50  0000 C CNN
+F 2 "Connector_PinHeader_2.54mm:PinHeader_1x05_P2.54mm_Vertical" H 7650 3150 50  0001 C CNN
+F 3 "~" H 7650 3150 50  0001 C CNN
+	1    7650 3150
+	1    0    0    -1
+$EndComp
+$Comp
+L Connector:Conn_01x05_Male VUVs1
+U 1 1 5FE2A087
 P 7600 3150
-F 0 "VU-LEDs1" H 7572 3032 50  0000 R CNN
-F 1 "Conn_01x04_Male" H 7572 3123 50  0000 R CNN
-F 2 "Connector_PinHeader_2.54mm:PinHeader_1x04_P2.54mm_Vertical" H 7600 3150 50  0001 C CNN
+F 0 "VUVs1" H 7572 3082 50  0000 R CNN
+F 1 "Conn_01x05_Male" H 7572 3173 50  0000 R CNN
+F 2 "Connector_PinHeader_2.54mm:PinHeader_1x05_P2.54mm_Vertical" H 7600 3150 50  0001 C CNN
 F 3 "~" H 7600 3150 50  0001 C CNN
 	1    7600 3150
 	-1   0    0    1
 $EndComp
+Wire Wire Line
+	7400 2950 7400 3050
+Connection ~ 7400 3050
+Wire Wire Line
+	7400 3050 7400 3150
+Connection ~ 7400 3150
+Wire Wire Line
+	7400 3150 7400 3250
+Connection ~ 7400 3250
+Wire Wire Line
+	7400 3250 7400 3350
+Connection ~ 7850 3350
+Wire Wire Line
+	7850 3350 7850 3750
+Connection ~ 7850 1650
+Wire Wire Line
+	7850 1650 7850 2150
+Connection ~ 7850 2150
+Wire Wire Line
+	7850 2150 7850 2250
+Connection ~ 7850 2250
+Wire Wire Line
+	7850 2250 7850 2350
+Connection ~ 7850 2350
+Wire Wire Line
+	7850 2350 7850 2450
+Connection ~ 7850 2450
+Wire Wire Line
+	7850 2450 7850 2550
+Connection ~ 7850 2550
+Wire Wire Line
+	7850 2550 7850 2950
+Connection ~ 7850 2950
+Wire Wire Line
+	7850 2950 7850 3050
+Connection ~ 7850 3050
+Wire Wire Line
+	7850 3050 7850 3150
+Connection ~ 7850 3150
+Wire Wire Line
+	7850 3150 7850 3250
+Connection ~ 7850 3250
+Wire Wire Line
+	7850 3250 7850 3350
+Connection ~ 7400 3350
+Wire Wire Line
+	2400 900  2400 4000
+Wire Wire Line
+	2400 4000 4300 4000
+Wire Wire Line
+	4150 3250 4150 3650
+Wire Wire Line
+	4150 3650 7400 3650
+Wire Wire Line
+	7400 3350 7400 3650
+Wire Wire Line
+	4050 3250 4050 3600
+Wire Wire Line
+	4050 3600 7300 3600
+Wire Wire Line
+	7300 3600 7300 2550
+Wire Wire Line
+	7300 2550 7400 2550
+Wire Wire Line
+	7400 2450 7250 2450
+Wire Wire Line
+	7250 2450 7250 3550
+Wire Wire Line
+	7250 3550 3950 3550
+Wire Wire Line
+	3950 3550 3950 3250
+Wire Wire Line
+	3850 3250 3850 3500
+Wire Wire Line
+	3850 3500 7150 3500
+Wire Wire Line
+	7150 3500 7150 2350
+Wire Wire Line
+	7150 2350 7400 2350
+Wire Wire Line
+	7400 2250 7100 2250
+Wire Wire Line
+	7100 2250 7100 3450
+Wire Wire Line
+	7100 3450 3750 3450
+Wire Wire Line
+	3750 3450 3750 3250
+Wire Wire Line
+	3650 3250 3650 3400
+Wire Wire Line
+	3650 3400 7050 3400
+Wire Wire Line
+	7050 3400 7050 2150
+Wire Wire Line
+	7050 2150 7400 2150
 $EndSCHEMATC

Commit message: 1st Controller_Mixer pcb fertig
Parts:
- added R1, R2, R3, R4, R5: R_PHOTO, Resistor_THT:R_Axial_DIN0207_L6.3mm_D2.5mm_P5.08mm_Vertical, symbol Device:R_PHOTO
Connections:
- net at U3.16 (24_A10_TX6_SCL2): now also R5.1; no longer LEDs1.1 (Pin_1)
- net at U3.30 (38_CS1_IN1): now also R4.1; no longer LEDs1.2 (Pin_2)
- net at U3.31 (39_MISO1_OUT1A): now also R3.1; no longer LEDs1.3 (Pin_3)
- net at U3.32 (40_A16): now also R2.1; no longer LEDs1.4 (Pin_4)
- net at U3.33 (41_A17): now also R1.1; no longer LEDs1.5 (Pin_5)
- new net: LEDs1.5 (Pin_5), R1.2
- new net: LEDs1.4 (Pin_4), R2.2
- new net: LEDs1.3 (Pin_3), R3.2
- new net: LEDs1.2 (Pin_2), R4.2
- new net: LEDs1.1 (Pin_1), R5.2
Other:
- moved on the sheet: J15, LEDs1
Changed lines of the file:
@@
 Wire Wire Line
 	1950 5600 1950 700
-Text GLabel 7950 550  3    50   UnSpc ~ 0
+Text GLabel 8450 550  3    50   UnSpc ~ 0
 LED-Connectors
 Text GLabel 7950 1300 3    50   UnSpc ~ 0
@@
 	7350 550  7350 650
 Wire Wire Line
-	7350 650  7400 650
-Wire Wire Line
 	4450 600  7300 600
 Wire Wire Line
 	7300 600  7300 750
 Wire Wire Line
-	7300 750  7400 750
-Wire Wire Line
 	4550 650  7250 650
 Wire Wire Line
 	7250 650  7250 850
 Wire Wire Line
-	7250 850  7400 850
-Wire Wire Line
 	7200 3700 7200 950
 Wire Wire Line
-	7200 950  7400 950
+	7700 950  7900 950
 Wire Wire Line
 	4250 3700 7200 3700
 Wire Wire Line
-	7850 550  7850 650
-Connection ~ 7850 650
-Wire Wire Line
-	7850 650  7850 750
-Connection ~ 7850 750
-Wire Wire Line
-	7850 750  7850 850
-Connection ~ 7850 850
-Wire Wire Line
-	7850 850  7850 950
-Connection ~ 7850 950
+	8350 550  8350 650
+Connection ~ 8350 650
+Wire Wire Line
+	8350 650  8350 750
+Connection ~ 8350 750
+Wire Wire Line
+	8350 750  8350 850
+Connection ~ 8350 850
+Wire Wire Line
+	8350 850  8350 950
+Connection ~ 8350 950
 Connection ~ 7850 1450
 Wire Wire Line
@@
 L Connector:Conn_01x05_Male J15
 U 1 1 5FA665C1
-P 7650 750
-F 0 "J15" H 7758 1131 50  0000 C CNN
-F 1 "Conn_01x05_Male" H 7758 1040 50  0000 C CNN
-F 2 "Connector_PinHeader_2.54mm:PinHeader_1x05_P2.54mm_Vertical" H 7650 750 50  0001 C CNN
-F 3 "~" H 7650 750 50  0001 C CNN
-	1    7650 750
+P 8150 750
+F 0 "J15" H 8258 1131 50  0000 C CNN
+F 1 "Conn_01x05_Male" H 8258 1040 50  0000 C CNN
+F 2 "Connector_PinHeader_2.54mm:PinHeader_1x05_P2.54mm_Vertical" H 8150 750 50  0001 C CNN
+F 3 "~" H 8150 750 50  0001 C CNN
+	1    8150 750
 	1    0    0    -1
 $EndComp
 Wire Wire Line
-	7850 950  7850 1250
+	8350 950  8350 1250
 $Comp
 L Connector:Conn_01x05_Male LEDs1
 U 1 1 5FA69E13
-P 7600 750
-F 0 "LEDs1" H 7572 682 50  0000 R CNN
-F 1 "Conn_01x05_Male" H 7572 773 50  0000 R CNN
-F 2 "Connector_PinHeader_2.54mm:PinHeader_1x05_P2.54mm_Vertical" H 7600 750 50  0001 C CNN
-F 3 "~" H 7600 750 50  0001 C CNN
-	1    7600 750
+P 8100 750
+F 0 "LEDs1" H 8072 682 50  0000 R CNN
+F 1 "Conn_01x05_Male" H 8072 773 50  0000 R CNN
+F 2 "Connector_PinHeader_2.54mm:PinHeader_1x05_P2.54mm_Vertical" H 8100 750 50  0001 C CNN
+F 3 "~" H 8100 750 50  0001 C CNN
+	1    8100 750
 	-1   0    0    1
 $EndComp
 Wire Wire Line
 	7850 1250 7850 1350
-Connection ~ 7850 1250
 Connection ~ 7850 1350
 Wire Wire Line
@@
 Wire Wire Line
 	7050 2150 7400 2150
+$Comp
+L Device:R_PHOTO R1
+U 1 1 5F92DF7D
+P 7550 550
+F 0 "R1" V 7757 550 50  0000 C CNN
+F 1 "R_PHOTO" V 7666 550 50  0000 C CNN
+F 2 "Resistor_THT:R_Axial_DIN0207_L6.3mm_D2.5mm_P5.08mm_Vertical" V 7600 300 50  0001 L CNN
+F 3 "~" H 7550 500 50  0001 C CNN
+	1    7550 550
+	0    -1   -1   0
+$EndComp
+$Comp
+L Device:R_PHOTO R2
+U 1 1 5F96E19E
+P 7550 650
+F 0 "R2" V 7757 650 50  0000 C CNN
+F 1 "R_PHOTO" V 7666 650 50  0000 C CNN
+F 2 "Resistor_THT:R_Axial_DIN0207_L6.3mm_D2.5mm_P5.08mm_Vertical" V 7600 400 50  0001 L CNN
+F 3 "~" H 7550 600 50  0001 C CNN
+	1    7550 650
+	0    -1   -1   0
+$EndComp
+$Comp
+L Device:R_PHOTO R3
+U 1 1 5F97B054
+P 7550 750
+F 0 "R3" V 7757 750 50  0000 C CNN
+F 1 "R_PHOTO" V 7666 750 50  0000 C CNN
+F 2 "Resistor_THT:R_Axial_DIN0207_L6.3mm_D2.5mm_P5.08mm_Vertical" V 7600 500 50  0001 L CNN
+F 3 "~" H 7550 700 50  0001 C CNN
+	1    7550 750
+	0    -1   -1   0
+$EndComp
+$Comp
+L Device:R_PHOTO R4
+U 1 1 5F987FB9
+P 7550 850
+F 0 "R4" V 7757 850 50  0000 C CNN
+F 1 "R_PHOTO" V 7666 850 50  0000 C CNN
+F 2 "Resistor_THT:R_Axial_DIN0207_L6.3mm_D2.5mm_P5.08mm_Vertical" V 7600 600 50  0001 L CNN
+F 3 "~" H 7550 800 50  0001 C CNN
+	1    7550 850
+	0    -1   -1   0
+$EndComp
+$Comp
+L Device:R_PHOTO R5
+U 1 1 5F994DBD
+P 7550 950
+F 0 "R5" V 7757 950 50  0000 C CNN
+F 1 "R_PHOTO" V 7666 950 50  0000 C CNN
+F 2 "Resistor_THT:R_Axial_DIN0207_L6.3mm_D2.5mm_P5.08mm_Vertical" V 7600 700 50  0001 L CNN
+F 3 "~" H 7550 900 50  0001 C CNN
+	1    7550 950
+	0    -1   -1   0
+$EndComp
+Wire Wire Line
+	7350 650  7400 650
+Wire Wire Line
+	7300 750  7400 750
+Wire Wire Line
+	7250 850  7400 850
+Wire Wire Line
+	7200 950  7400 950
+Wire Wire Line
+	7700 850  7900 850
+Wire Wire Line
+	7700 750  7900 750
+Wire Wire Line
+	7700 650  7900 650
+Wire Wire Line
+	7700 550  7900 550
+Wire Wire Line
+	7850 1250 8350 1250
+Connection ~ 7850 1250
 $EndSCHEMATC

Commit message: daily edits
Parts:
- added A5-1, A5-9: Conn_01x05_Male, Connector_PinHeader_2.54mm:PinHeader_1x05_P2.54mm_Vertical, symbol Connector:Conn_01x05_Male
- added D0-7, J12: Conn_01x08_Male, Connector_PinHeader_2.54mm:PinHeader_1x08_P2.54mm_Vertical, symbol Connector:Conn_01x08_Male
- added J11: USB_B, Connector_USB:USB_B_Lumberg_2411_02_Horizontal, symbol Connector:USB_B
Connections:
- net at VUVs1.1 (Pin_1), VUVs1.2 (Pin_2), VUVs1.3 (Pin_3)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: now also U3.48 (VIN), U3.49 (VUSB), J11.1 (VBUS); no longer U3.15 (3V3)
- net at U3.2 (0_RX1_CRX2_CS1): now also D0-7.1 (Pin_1)
- net at U3.3 (1_TX1_CTX2_MISO1): now also D0-7.2 (Pin_2)
- net at U3.4 (2_OUT2): now also D0-7.3 (Pin_3)
- net at U3.41 (19_A5_SCL): now also A5-9.1 (Pin_1)
- net at U3.42 (20_A6_TX5_LRCLK1): now also A5-9.2 (Pin_2)
- net at U3.43 (21_A7_RX5_BCLK1): now also A5-9.3 (Pin_3)
- net at U3.44 (22_A8_CTX1): now also A5-9.4 (Pin_4)
- net at U3.45 (23_A9_CRX1_MCLK1): now also A5-9.5 (Pin_5)
- net at U3.47 (GND): now also A5-1.1 (Pin_1), A5-1.2 (Pin_2), A5-1.3 (Pin_3), A5-1.4 (Pin_4), A5-1.5 (Pin_5), J11.4 (GND), J11.5 (Shield), J12.1 (Pin_1), J12.2 (Pin_2), J12.3 (Pin_3), J12.4 (Pin_4), J12.5 (Pin_5), J12.6 (Pin_6), J12.7 (Pin_7), J12.8 (Pin_8)
- net at U3.5 (3_LRCLK2): now also D0-7.4 (Pin_4)
- net at U3.6 (4_BCLK2): now also D0-7.5 (Pin_5)
- net at U3.66 (D-): now also J11.2 (D-)
- net at U3.67 (D+): now also J11.3 (D+)
- net at U3.7 (5_IN2): now also D0-7.6 (Pin_6)
- net at U3.8 (6_OUT1D): now also D0-7.7 (Pin_7)
- net at U3.9 (7_RX2_OUT1A): now also D0-7.8 (Pin_8)
Changed lines of the file:
@@
 	3750 650  1900 650
-Wire Wire Line
-	1850 600  3850 600
 Wire Wire Line
 	3950 550  1800 550
@@
 $EndComp
 $Comp
-L teensy:Teensy4.1 U3
-U 1 1 5F9167EF
-P 4900 2150
-F 0 "U3" V 4854 4578 50  0000 L CNN
-F 1 "Teensy4.1" V 4945 4578 50  0000 L CNN
-F 2 "Teensy:Teensy41" H 4500 2550 50  0001 C CNN
-F 3 "" H 4500 2550 50  0001 C CNN
-	1    4900 2150
-	0    -1   -1   0
-$EndComp
-$Comp
 L Connector:Conn_01x05_Male J15
 U 1 1 5FA665C1
@@
 	7850 1350 7850 1450
 Wire Wire Line
-	2400 900  2950 900
-Wire Wire Line
 	2950 900  2950 1050
 $Comp
@@
 Wire Wire Line
 	7850 3250 7850 3350
-Connection ~ 7400 3350
 Wire Wire Line
 	2400 900  2400 4000
 Wire Wire Line
 	2400 4000 4300 4000
-Wire Wire Line
-	4150 3250 4150 3650
-Wire Wire Line
-	4150 3650 7400 3650
-Wire Wire Line
-	7400 3350 7400 3650
 Wire Wire Line
 	4050 3250 4050 3600
@@
 	7850 1250 8350 1250
 Connection ~ 7850 1250
+$Comp
+L teensy:Teensy4.1 U3
+U 1 1 5F9167EF
+P 4900 2150
+F 0 "U3" V 4854 4578 50  0000 L CNN
+F 1 "Teensy4.1" V 4945 4578 50  0000 L CNN
+F 2 "Teensy:Teensy41" H 4500 2550 50  0001 C CNN
+F 3 "" H 4500 2550 50  0001 C CNN
+	1    4900 2150
+	0    -1   -1   0
+$EndComp
+$Comp
+L Connector:USB_B J11
+U 1 1 5F9CE4FA
+P 1450 1550
+F 0 "J11" H 1507 2017 50  0000 C CNN
+F 1 "USB_B" H 1507 1926 50  0000 C CNN
+F 2 "Connector_USB:USB_B_Lumberg_2411_02_Horizontal" H 1600 1500 50  0001 C CNN
+F 3 " ~" H 1600 1500 50  0001 C CNN
+	1    1450 1550
+	1    0    0    -1
+$EndComp
+Wire Wire Line
+	1450 1950 1350 1950
+Wire Wire Line
+	1200 850  2850 850
+Wire Wire Line
+	2850 850  2850 1050
+Connection ~ 1350 1950
+Wire Wire Line
+	1350 1950 1200 1950
+Wire Wire Line
+	2400 900  2950 900
+Wire Wire Line
+	1750 1350 1750 950
+Wire Wire Line
+	1750 950  2250 950
+Wire Wire Line
+	2750 950  2750 1050
+Wire Wire Line
+	1750 1550 2350 1550
+Wire Wire Line
+	2350 1550 2350 3350
+Wire Wire Line
+	2350 3350 5350 3350
+Wire Wire Line
+	5350 3350 5350 3250
+Wire Wire Line
+	1750 1650 2300 1650
+Wire Wire Line
+	2300 1650 2300 3300
+Wire Wire Line
+	2300 3300 5250 3300
+Wire Wire Line
+	5250 3300 5250 3250
+Wire Wire Line
+	7400 3350 7400 3650
+Wire Wire Line
+	7400 3650 2250 3650
+Wire Wire Line
+	2250 3650 2250 950
+Connection ~ 7400 3350
+Connection ~ 2250 950
+$Comp
+L Connector:Conn_01x08_Male D0-7
+U 1 1 5FCD0BE9
+P 3150 3450
+F 0 "D0-7" V 3077 3378 50  0000 C CNN
+F 1 "Conn_01x08_Male" V 2986 3378 50  0000 C CNN
+F 2 "Connector_PinHeader_2.54mm:PinHeader_1x08_P2.54mm_Vertical" H 3150 3450 50  0001 C CNN
+F 3 "~" H 3150 3450 50  0001 C CNN
+	1    3150 3450
+	0    -1   -1   0
+$EndComp
+Wire Wire Line
+	2250 950  2600 950
+Wire Wire Line
+	2600 1050 2600 950
+Connection ~ 2600 950
+Wire Wire Line
+	2600 950  2750 950
+Wire Wire Line
+	1850 600  3850 600
+$Comp
+L Connector:Conn_01x05_Male A5-9
+U 1 1 5FD59210
+P 3250 850
+F 0 "A5-9" V 3312 1094 50  0000 L CNN
+F 1 "Conn_01x05_Male" V 3403 1094 50  0000 L CNN
+F 2 "Connector_PinHeader_2.54mm:PinHeader_1x05_P2.54mm_Vertical" H 3250 850 50  0001 C CNN
+F 3 "~" H 3250 850 50  0001 C CNN
+	1    3250 850
+	0    1    1    0
+$EndComp
+$Comp
+L Connector:Conn_01x08_Male J12
+U 1 1 5FD968A0
+P 1000 2150
+F 0 "J12" V 927 2078 50  0000 C CNN
+F 1 "Conn_01x08_Male" V 836 2078 50  0000 C CNN
+F 2 "Connector_PinHeader_2.54mm:PinHeader_1x08_P2.54mm_Vertical" H 1000 2150 50  0001 C CNN
+F 3 "~" H 1000 2150 50  0001 C CNN
+	1    1000 2150
+	1    0    0    -1
+$EndComp
+$Comp
+L Connector:Conn_01x05_Male A5-1
+U 1 1 5FDAA8DC
+P 1000 1550
+F 0 "A5-1" V 1062 1794 50  0000 L CNN
+F 1 "Conn_01x05_Male" V 1153 1794 50  0000 L CNN
+F 2 "Connector_PinHeader_2.54mm:PinHeader_1x05_P2.54mm_Vertical" H 1000 1550 50  0001 C CNN
+F 3 "~" H 1000 1550 50  0001 C CNN
+	1    1000 1550
+	1    0    0    -1
+$EndComp
+Wire Wire Line
+	1200 850  1200 1350
+Connection ~ 1200 1350
+Wire Wire Line
+	1200 1350 1200 1450
+Connection ~ 1200 1450
+Wire Wire Line
+	1200 1450 1200 1550
+Connection ~ 1200 1550
+Wire Wire Line
+	1200 1550 1200 1650
+Connection ~ 1200 1650
+Wire Wire Line
+	1200 1650 1200 1750
+Connection ~ 1200 1750
+Wire Wire Line
+	1200 1750 1200 1850
+Wire Wire Line
+	1200 1750 1200 1850
+Connection ~ 1200 1850
+Wire Wire Line
+	1200 1850 1200 1950
+Connection ~ 1200 1950
+Wire Wire Line
+	1200 1950 1200 2050
+Connection ~ 1200 2050
+Wire Wire Line
+	1200 2050 1200 2150
+Connection ~ 1200 2150
+Wire Wire Line
+	1200 2150 1200 2250
+Connection ~ 1200 2250
+Wire Wire Line
+	1200 2250 1200 2350
+Connection ~ 1200 2350
+Wire Wire Line
+	1200 2350 1200 2450
+Connection ~ 1200 2450
+Wire Wire Line
+	1200 2450 1200 2550
 $EndSCHEMATC

Commit message: diesdas
Parts:
- added C1: CP1_Small, Capacitor_THT:CP_Axial_L10.0mm_D4.5mm_P15.00mm_Horizontal, symbol Device:CP1_Small
- added J13: RJ45_Amphenol_RJMG1BD3B8K1ANR, Connector_RJ:RJ45_Amphenol_RJMG1BD3B8K1ANR, symbol Connector:RJ45_Amphenol_RJMG1BD3B8K1ANR
Connections:
- net at R+|LED|T-1.1 (Pin_1), U3.60 (R+): now also J13.R3 (RD+)
- net at R+|LED|T-1.2 (Pin_2), U3.61 (LED): now also J13.L4 (LEDG_A)
- net at R+|LED|T-1.3 (Pin_3), U3.62 (T-): now also J13.R2 (TD-)
- net at T+|GND|R-1.1 (Pin_1), U3.63 (T+): now also J13.R1 (TD+)
- net at T+|GND|R-1.2 (Pin_2), U3.64 (GND): now also C1.2, J13.L3 (LEDG_K), J13.R8 (GND)
- net at T+|GND|R-1.3 (Pin_3), U3.65 (R-): now also J13.R6 (RD-)
- new net: C1.1, J13.R4 (TCT), J13.R5 (RCT)
Other:
- moved on the sheet: R+|LED|T-1, T+|GND|R-1
Changed lines of the file:
@@
 L Connector:Conn_01x03_Male T+|GND|R-1
 U 1 1 5FABE9C0
-P 5400 850
-F 0 "T+|GND|R-1" V 5462 994 50  0000 L CNN
-F 1 "Conn_01x03_Male" V 5553 994 50  0000 L CNN
-F 2 "Connector_PinHeader_2.54mm:PinHeader_1x03_P2.54mm_Vertical" H 5400 850 50  0001 C CNN
-F 3 "~" H 5400 850 50  0001 C CNN
-	1    5400 850
+P 8250 1450
+F 0 "T+|GND|R-1" V 8312 1594 50  0000 L CNN
+F 1 "Conn_01x03_Male" V 8403 1594 50  0000 L CNN
+F 2 "Connector_PinHeader_2.54mm:PinHeader_1x03_P2.54mm_Vertical" H 8250 1450 50  0001 C CNN
+F 3 "~" H 8250 1450 50  0001 C CNN
+	1    8250 1450
 	0    1    1    0
 $EndComp
@@
 L Connector:Conn_01x03_Male R+|LED|T-1
 U 1 1 5FAC1385
-P 5700 850
-F 0 "R+|LED|T-1" V 5762 994 50  0000 L CNN
-F 1 "Conn_01x03_Male" V 5853 994 50  0000 L CNN
-F 2 "Connector_PinHeader_2.54mm:PinHeader_1x03_P2.54mm_Vertical" H 5700 850 50  0001 C CNN
-F 3 "~" H 5700 850 50  0001 C CNN
-	1    5700 850
+P 8550 1450
+F 0 "R+|LED|T-1" V 8612 1594 50  0000 L CNN
+F 1 "Conn_01x03_Male" V 8703 1594 50  0000 L CNN
+F 2 "Connector_PinHeader_2.54mm:PinHeader_1x03_P2.54mm_Vertical" H 8550 1450 50  0001 C CNN
+F 3 "~" H 8550 1450 50  0001 C CNN
+	1    8550 1450
 	0    1    1    0
 $EndComp
@@
 Wire Wire Line
 	1200 1750 1200 1850
-Wire Wire Line
-	1200 1750 1200 1850
 Connection ~ 1200 1850
 Wire Wire Line
@@
 Wire Wire Line
 	1200 2450 1200 2550
+$Comp
+L Connector:RJ45_Amphenol_RJMG1BD3B8K1ANR J13
+U 1 1 5F9D8B7C
+P 9850 2700
+F 0 "J13" H 9850 3425 50  0000 C CNN
+F 1 "RJ45_Amphenol_RJMG1BD3B8K1ANR" H 9850 3334 50  0000 C CNN
+F 2 "Connector_RJ:RJ45_Amphenol_RJMG1BD3B8K1ANR" H 9850 3400 50  0001 C CNN
+F 3 "https://www.amphenolcanada.com/ProductSearch/Drawings/AC/RJMG1BD3B8K1ANR.PDF" H 9850 3500 50  0001 C CNN
+	1    9850 2700
+	1    0    0    -1
+$EndComp
+Wire Wire Line
+	5500 1050 5500 1700
+Wire Wire Line
+	5500 1700 8350 1700
+Wire Wire Line
+	8350 1700 8350 1650
+Wire Wire Line
+	8350 1700 8350 2200
+Wire Wire Line
+	8350 2200 8950 2200
+Connection ~ 8350 1700
+Wire Wire Line
+	5600 1050 5600 1750
+Wire Wire Line
+	5600 1750 8450 1750
+Wire Wire Line
+	8450 1750 8450 1650
+Wire Wire Line
+	8450 1750 8450 2400
+Wire Wire Line
+	8450 2400 8950 2400
+Connection ~ 8450 1750
+Wire Wire Line
+	5400 1050 5400 1800
+Wire Wire Line
+	5400 1800 8250 1800
+Wire Wire Line
+	8250 1800 8250 1650
+Wire Wire Line
+	8250 3400 8800 3400
+Connection ~ 8250 1800
+Wire Wire Line
+	8950 3000 8250 3000
+Connection ~ 8250 3000
+Wire Wire Line
+	8250 3000 8250 3400
+Wire Wire Line
+	5300 1050 5300 1900
+Wire Wire Line
+	5300 1900 8150 1900
+Wire Wire Line
+	8150 1900 8150 1650
+Wire Wire Line
+	8150 1900 8150 2700
+Wire Wire Line
+	8150 2700 8950 2700
+Connection ~ 8150 1900
+Wire Wire Line
+	8250 1800 8250 3000
+Wire Wire Line
+	5700 1050 5700 1950
+Wire Wire Line
+	5700 1950 8550 1950
+Wire Wire Line
+	8550 1950 8550 1650
+Wire Wire Line
+	8550 1950 8550 2900
+Wire Wire Line
+	8550 2900 8950 2900
+Connection ~ 8550 1950
+Wire Wire Line
+	5800 1050 5800 2050
+Wire Wire Line
+	5800 2050 8650 2050
+Wire Wire Line
+	8650 2050 8650 1650
+Wire Wire Line
+	8650 2050 8650 2500
+Wire Wire Line
+	8650 2500 8950 2500
+Connection ~ 8650 2050
+$Comp
+L Device:CP1_Small C1
+U 1 1 5FB5EC34
+P 8800 3200
+F 0 "C1" H 8891 3246 50  0000 L CNN
+F 1 "CP1_Small" H 8891 3155 50  0000 L CNN
+F 2 "Capacitor_THT:CP_Axial_L10.0mm_D4.5mm_P15.00mm_Horizontal" H 8800 3200 50  0001 C CNN
+F 3 "~" H 8800 3200 50  0001 C CNN
+	1    8800 3200
+	1    0    0    -1
+$EndComp
+Wire Wire Line
+	8950 2300 8800 2300
+Wire Wire Line
+	8800 2300 8800 2600
+Wire Wire Line
+	8950 2600 8800 2600
+Connection ~ 8800 2600
+Wire Wire Line
+	8800 2600 8800 3100
+Wire Wire Line
+	8800 3300 8800 3400
+Connection ~ 8800 3400
+Wire Wire Line
+	8800 3400 9850 3400
 $EndSCHEMATC
