File: Controller_Mixer/pcb/controller_mixer_pcb_v0.2/mixer.pcb.sch (KiCad schematic (older format))
At the start: 78 parts, among them J1 Conn_01x03, J10 Conn_01x02, J11 Conn_01x02, J12 Conn_01x02, J13 Conn_01x02, J14 Conn_01x02, J15 Conn_01x02, J16 Conn_01x02, J2 Conn_01x03, J3 Conn_01x03, J4 Conn_01x03, J41 Conn_01x04, J42 Conn_01x04, J43 Conn_01x03, J44 Conn_01x02, J45 Conn_01x02, J46 Conn_01x02, J47 Conn_01x02, J48 Conn_01x02, J49 Conn_01x02, J5 Conn_01x03, J50 Conn_01x02, J51 Conn_01x02, J52 Conn_01x02, J53 Conn_01x02, J54 Conn_01x05, J55 Conn_01x05, J56 Conn_01x05, J57 Conn_01x05, J58 Conn_01x05, J59 Conn_01x05, J6 Conn_01x03, J7 Conn_01x03, J71 Conn_01x03, J72 Conn_01x03, J8 Conn_01x03, J9 Conn_01x02, U1 74HC4051, U3 74HC4051, U5 Teensy4.1, U8 74HC4051

Commit message: mixer pcb v0.2 ready?
Parts:
- MuxCh1_1: renamed from J?; Field4 (none) -> MuxCh1_1
- MuxCh1_2: renamed from J?; Field4 (none) -> MuxCh1_2
- MuxCh1_3: renamed from J?; Field4 (none) -> MuxCh1_3
- MuxCh1_4: renamed from J?; Field4 (none) -> MuxCh1_4
- MuxCh1_5: renamed from J?; Field4 (none) -> MuxCh1_5
- MuxCh1_6: renamed from J?; Field4 (none) -> MuxCh1_6
- MuxCh1_7: renamed from J?; Field4 (none) -> MuxCh1_7
- MuxCh1_8: renamed from J?; Field4 (none) -> MuxCh1_8
- MuxCh2_1: renamed from J?; Field4 (none) -> MuxCh2_1
- MuxCh2_2: renamed from J?; Field4 (none) -> MuxCh2_2
- MuxCh2_3: renamed from J?; Field4 (none) -> MuxCh2_3
- MuxCh2_4: renamed from J?; Field4 (none) -> MuxCh2_4
- MuxCh2_5: renamed from J?; Field4 (none) -> MuxCh2_5
- MuxCh2_6: renamed from J?; Field4 (none) -> MuxCh2_6
- MuxCh2_7: renamed from J?; Field4 (none) -> MuxCh2_7
- MuxCh2_8: renamed from J?; Field4 (none) -> MuxCh2_8
- MuxCh3_1: renamed from J1; Field4 (none) -> MuxCh3_1
- MuxCh3_2: renamed from J2; Field4 (none) -> MuxCh3_2
- MuxCh3_3: renamed from J3; Field4 (none) -> MuxCh3_3
- MuxCh3_4: renamed from J4; Field4 (none) -> MuxCh3_4
- MuxCh3_5: renamed from J5; Field4 (none) -> MuxCh3_5
- MuxCh3_6: renamed from J6; Field4 (none) -> MuxCh3_6
- MuxCh3_7: renamed from J7; Field4 (none) -> MuxCh3_7
- MuxCh3_8: renamed from J8; Field4 (none) -> MuxCh3_8
- MuxCh4_1: renamed from J?; Field4 (none) -> MuxCh4_1
- MuxCh4_2: renamed from J?; Field4 (none) -> MuxCh4_2
- MuxCh4_3: renamed from J?; Field4 (none) -> MuxCh4_3
- MuxCh4_4: renamed from J?; Field4 (none) -> MuxCh4_4
- MuxCh4_5: renamed from J?; Field4 (none) -> MuxCh4_5
- MuxCh4_6: renamed from J?; Field4 (none) -> MuxCh4_6
- MuxCh4_7: renamed from J?; Field4 (none) -> MuxCh4_7
- MuxCh4_8: renamed from J?; Field4 (none) -> MuxCh4_8
- MuxMaster_1: renamed from J?; Field4 (none) -> MuxMaster_1
- MuxMaster_2: renamed from J?; Field4 (none) -> MuxMaster_2
- MuxMaster_3: renamed from J?; Field4 (none) -> MuxMaster_3
- MuxMaster_4: renamed from J?; Field4 (none) -> MuxMaster_4
- MuxMaster_5: renamed from J?; Field4 (none) -> MuxMaster_5
- MuxMaster_6: renamed from J?; Field4 (none) -> MuxMaster_6
- MuxMaster_7: renamed from J?; Field4 (none) -> MuxMaster_7
- MuxMaster_8: renamed from J?; Field4 (none) -> MuxMaster_8
- NeoPixel1: renamed from J43; Field4 (none) -> NeoPixel
- VU_Matrix1: renamed from J?; footprint (none) -> Connector_JST:JST_XH_B5B-XH-A_1x05_P2.50mm_Vertical; Field4 (none) -> VU_Matrix
- display_1: renamed from J42; Field4 (none) -> display_1
- display_2: renamed from J41; Field4 (none) -> display_2
- fx1_btn1: renamed from J9; Field4 (none) -> fx1_btn1
- fx1_btn2: renamed from J10; Field4 (none) -> fx1_btn2
- fx1_btn3: renamed from J11; Field4 (none) -> fx1_btn3
- fx1_btn4: renamed from J12; Field4 (none) -> fx1_btn4
- fx1_enc1: renamed from J54; Field4 (none) -> fx1_enc1
- fx1_enc2: renamed from J55; Field4 (none) -> fx1_enc2
- fx1_enc3: renamed from J56; Field4 (none) -> fx1_enc3
- fx2_btn1: renamed from J13; Field4 (none) -> fx2_btn1
- fx2_btn2: renamed from J14; Field4 (none) -> fx2_btn2
- fx2_btn3: renamed from J15; Field4 (none) -> fx2_btn3
- fx2_btn4: renamed from J16; Field4 (none) -> fx2_btn4
- fx2_enc1: renamed from J57; Field4 (none) -> fx2_enc1
- fx2_enc2: renamed from J58; Field4 (none) -> fx2_enc2
- fx2_enc3: renamed from J59; Field4 (none) -> fx2_enc3
- pfl_btn_1: renamed from J53; Field4 (none) -> pfl_btn_1
- pfl_btn_2: renamed from J52; Field4 (none) -> pfl_btn_2
- pfl_btn_3: renamed from J51; Field4 (none) -> pfl_btn_3
- pfl_btn_4: renamed from J50; Field4 (none) -> pfl_btn_4
- pfl_btn_master1: renamed from J49; Field4 (none) -> pfl_btn_master
- pfl_led_1: renamed from J48; Field4 (none) -> pfl_led_1
- pfl_led_2: renamed from J47; Field4 (none) -> pfl_led_2
- pfl_led_3: renamed from J46; Field4 (none) -> pfl_led_3
- pfl_led_4: renamed from J45; Field4 (none) -> pfl_led_4
- pfl_led_master1: renamed from J44; Field4 (none) -> pfl_led_master
- spare(28)1: renamed from J71; Field4 (none) -> spare(28)
- spare(29)1: renamed from J72; Field4 (none) -> spare(29)
- gave numbers to parts that had none: 4
- renumbered U3 to FX-BTNs1, U1 to MuxCh3, U8 to fxEncBtns1
Connections:
- net mux_ch1: now also MuxCh1.3 (A); no longer MuxCh3.3 (A)
- net mux_ch2: now also MuxCh2.3 (A); no longer MuxCh4.3 (A)
- net mux_ch3: now also MuxCh3.3 (A); no longer MuxCh2.3 (A)
- net mux_ch4: now also MuxCh4.3 (A); no longer MuxCh1.3 (A)
Other:
- moved on the sheet: MuxCh1, MuxCh1_1, MuxCh1_2, MuxCh1_3, MuxCh1_4, MuxCh1_5, MuxCh1_6, MuxCh1_7, MuxCh1_8, MuxCh2, MuxCh2_1, MuxCh2_2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

Commit message: mixer pcb
Parts:
- removed MuxCh2_1, MuxCh2_2, MuxCh2_3, MuxCh2_4, MuxCh2_5, MuxCh2_6, MuxCh2_7, MuxCh2_8, MuxCh3_1, MuxCh3_2, MuxCh3_3, MuxCh3_4, MuxCh3_5, MuxCh3_6, MuxCh3_7, MuxCh3_8, MuxCh4_1, MuxCh4_2, MuxCh4_3, MuxCh4_4, MuxCh4_5, MuxCh4_6, MuxCh4_7, MuxCh4_8, MuxMaster_1, MuxMaster_2, MuxMaster_3, MuxMaster_4, MuxMaster_5, MuxMaster_6, MuxMaster_7, MuxMaster_8: Conn_01x03, Connector_JST:JST_XH_B3B-XH-A_1x03_P2.50mm_Vertical, symbol Connector_Generic:Conn_01x03
- removed muxMaster1: 74HC4051, Package_DIP:DIP-16_W7.62mm, symbol 74xx:74HC4051
- added C1: CP, Capacitor_THT:CP_Radial_D10.0mm_P2.50mm, symbol mixer.pcb-rescue:CP-Device
- added MuxCh1_10, MuxCh1_11, MuxCh1_12, MuxCh1_13, MuxCh1_14, MuxCh1_15, MuxCh1_16, MuxCh1_17, MuxCh1_18, MuxCh1_19, MuxCh1_20, MuxCh1_21, MuxCh1_22, MuxCh1_23, MuxCh1_24, MuxCh1_25, MuxCh1_26, MuxCh1_27, MuxCh1_28, MuxCh1_29, MuxCh1_30, MuxCh1_31, MuxCh1_32, MuxCh1_33, MuxCh1_34, MuxCh1_35, MuxCh1_36, MuxCh1_37, MuxCh1_38, MuxCh1_39, MuxCh1_40, MuxCh1_9: Conn_01x03, Connector_JST:JST_XH_B3B-XH-A_1x03_P2.50mm_Vertical, symbol Connector_Generic:Conn_01x03
- added MuxCh5: 74HC4051, Package_DIP:DIP-16_W7.62mm, symbol 74xx:74HC4051
- added R1, R10, R11, R12, R13, R14, R15, R16, R17, R19, R2, R20, R21, R22, R23, R24, R25, R26, R27, R28, R29, R3, R34, R35, R36, R37, R38, R39, R4, R40, R41, R42, R43, R44, R45, R46, R47, R48, R49, R5, R50, R51, R52, R53, R54, R55, R56, R57, R58, R59, R6, R60, R61, R62, R63, R64, R65, R66, R67, R7, R8, R9: 100k, Resistor_THT:R_Axial_DIN0207_L6.3mm_D2.5mm_P10.16mm_Horizontal, symbol mixer.pcb-rescue:R-Device
- added R18, R30, R31, R32, R33: 500, Resistor_THT:R_Axial_DIN0207_L6.3mm_D2.5mm_P10.16mm_Horizontal, symbol mixer.pcb-rescue:R-Device
- VU_Matrix1: symbol mixer.pcb:Connector_Generic_Conn_01x05 -> mixer.pcb-rescue:Connector_Generic_Conn_01x05-mixer.pcb
Connections:
- net +3V3: now also C1.1, C1.2, MuxCh1_10.1 (Pin_1), MuxCh1_11.1 (Pin_1), MuxCh1_12.1 (Pin_1), MuxCh1_13.1 (Pin_1), MuxCh1_14.1 (Pin_1), MuxCh1_15.1 (Pin_1), MuxCh1_16.1 (Pin_1), MuxCh1_17.1 (Pin_1), MuxCh1_18.1 (Pin_1), MuxCh1_19.1 (Pin_1), MuxCh1_20.1 (Pin_1), MuxCh1_21.1 (Pin_1), MuxCh1_22.1 (Pin_1), MuxCh1_23.1 (Pin_1), MuxCh1_24.1 (Pin_1), MuxCh1_25.1 (Pin_1), MuxCh1_26.1 (Pin_1), MuxCh1_27.1 (Pin_1), MuxCh1_28.1 (Pin_1), MuxCh1_29.1 (Pin_1), MuxCh1_30.1 (Pin_1), MuxCh1_31.1 (Pin_1), MuxCh1_32.1 (Pin_1), MuxCh1_33.1 (Pin_1), MuxCh1_34.1 (Pin_1), MuxCh1_35.1 (Pin_1), MuxCh1_36.1 (Pin_1), MuxCh1_37.1 (Pin_1), MuxCh1_38.1 (Pin_1), MuxCh1_39.1 (Pin_1), MuxCh1_40.1 (Pin_1), MuxCh1_9.1 (Pin_1), MuxCh5.16 (VCC)
- net GND: now also MuxCh1_10.3 (Pin_3), MuxCh1_11.3 (Pin_3), MuxCh1_12.3 (Pin_3), MuxCh1_13.3 (Pin_3), MuxCh1_14.3 (Pin_3), MuxCh1_15.3 (Pin_3), MuxCh1_16.3 (Pin_3), MuxCh1_17.3 (Pin_3), MuxCh1_18.3 (Pin_3), MuxCh1_19.3 (Pin_3), MuxCh1_20.3 (Pin_3), MuxCh1_21.3 (Pin_3), MuxCh1_22.3 (Pin_3), MuxCh1_23.3 (Pin_3), MuxCh1_24.3 (Pin_3), MuxCh1_25.3 (Pin_3), MuxCh1_26.3 (Pin_3), MuxCh1_27.3 (Pin_3), MuxCh1_28.3 (Pin_3), MuxCh1_29.3 (Pin_3), MuxCh1_30.3 (Pin_3), MuxCh1_31.3 (Pin_3), MuxCh1_32.3 (Pin_3), MuxCh1_33.3 (Pin_3), MuxCh1_34.3 (Pin_3), MuxCh1_35.3 (Pin_3), MuxCh1_36.3 (Pin_3), MuxCh1_37.3 (Pin_3), MuxCh1_38.3 (Pin_3), MuxCh1_39.3 (Pin_3), MuxCh1_40.3 (Pin_3), MuxCh1_9.3 (Pin_3), MuxCh5.6 (~E), MuxCh5.7 (VEE), MuxCh5.8 (GND), R1.2, R10.2, R11.2, R12.2, R13.2, R14.2, R15.2, R16.2, R17.2, R19.2, R2.2, R20.2, R21.2, R22.2, R23.2, R24.2, R25.2, R26.2, R27.2, R28.2, R29.2, R3.2, R34.2, R35.2, R36.2, R37.2, R38.2, R39.2, R4.2, R40.2, R41.2, R42.2, R43.2, R44.2, R45.2, R46.2, R47.2, R48.2, R49.2, R5.2, R50.2, R51.2, R52.2, R53.2, R54.2, R55.2, R56.2, R57.2, R58.2, R59.2, R6.2, R60.2, R61.2, R62.2, R63.2, R64.2, R65.2, R66.2, R67.2, R7.2, R8.2, R9.2
- net mux_ch1: now also R38.1
- net mux_ch2: now also R37.1
- net mux_ch3: now also R36.1
- net mux_ch4: now also R35.1
- net mux_encBtn_fx: now also R17.1
- net mux_master: now also MuxCh5.3 (A), R34.1
- net mux_selBtn_fx: now also R19.1
- net pfl_btn_ch1: now also R43.1
- net pfl_btn_ch2: now also R42.1
- net pfl_btn_ch3: now also R41.1
- net pfl_btn_ch4: now also R40.1
- net pfl_btn_master: now also R39.1
- net pfl_led_ch1: now also R18.2; no longer U5.18 (26_A12_MOSI1)
- net pfl_led_ch2: now also R33.1; no longer U5.30 (38_CS1_IN1)
- net pfl_led_ch3: now also R32.1; no longer U5.31 (39_MISO1_OUT1A)
- net pfl_led_ch4: now also R31.1; no longer U5.32 (40_A16)
- net pfl_led_master: now also R30.1; no longer U5.33 (41_A17)
- net pin28: now also R20.1
- net pin29: now also R21.1
- net s0: now also MuxCh5.11 (S0)
- net s1: now also MuxCh5.10 (S1)
- net s2: now also MuxCh5.9 (S2)
- net at MuxCh3.1 (A4): now also MuxCh1_21.2 (Pin_2), R48.1
- net at MuxCh3.12 (A3): now also MuxCh1_20.2 (Pin_2), R47.1
- net at MuxCh3.13 (A0): now also MuxCh1_17.2 (Pin_2), R44.1
- net at MuxCh3.14 (A1): now also MuxCh1_18.2 (Pin_2), R45.1
- net at MuxCh3.15 (A2): now also MuxCh1_19.2 (Pin_2), R46.1
- net at MuxCh3.2 (A6): now also MuxCh1_23.2 (Pin_2), R50.1
- net at MuxCh3.4 (A7): now also MuxCh1_24.2 (Pin_2), R51.1
- net at MuxCh3.5 (A5): now also MuxCh1_22.2 (Pin_2), R49.1
- net at MuxCh4.2 (A6): now also MuxCh1_31.2 (Pin_2), R58.1
- net at MuxCh4.12 (A3): now also MuxCh1_28.2 (Pin_2), R55.1
- net at MuxCh4.15 (A2): now also MuxCh1_27.2 (Pin_2), R54.1
- net at MuxCh4.14 (A1): now also MuxCh1_26.2 (Pin_2), R53.1
- net at MuxCh4.4 (A7): now also MuxCh1_32.2 (Pin_2), R59.1
- net at MuxCh4.5 (A5): now also MuxCh1_30.2 (Pin_2), R57.1
- net at MuxCh4.1 (A4): now also MuxCh1_29.2 (Pin_2), R56.1
- net at MuxCh4.13 (A0): now also MuxCh1_25.2 (Pin_2), R52.1
- net at MuxCh2.2 (A6): now also MuxCh1_15.2 (Pin_2), R28.1
- net at MuxCh2.12 (A3): now also MuxCh1_12.2 (Pin_2), R25.1
- net at MuxCh2.15 (A2): now also MuxCh1_11.2 (Pin_2), R24.1
- net at MuxCh2.14 (A1): now also MuxCh1_10.2 (Pin_2), R23.1
- net at MuxCh2.4 (A7): now also MuxCh1_16.2 (Pin_2), R29.1
- net at MuxCh2.5 (A5): now also MuxCh1_14.2 (Pin_2), R27.1
- net at MuxCh2.1 (A4): now also MuxCh1_13.2 (Pin_2), R26.1
- net at MuxCh2.13 (A0): now also MuxCh1_9.2 (Pin_2), R22.1
- net at MuxCh1.2 (A6), MuxCh1_7.2 (Pin_2): now also R15.1
- net at MuxCh1.12 (A3), MuxCh1_4.2 (Pin_2): now also R12.1
- net at MuxCh1.15 (A2), MuxCh1_3.2 (Pin_2): now also R11.1
- net at MuxCh1.14 (A1), MuxCh1_2.2 (Pin_2): now also R10.1
- net at MuxCh1.4 (A7), MuxCh1_8.2 (Pin_2): now also R16.1
- net at MuxCh1.5 (A5), MuxCh1_6.2 (Pin_2): now also R14.1
- net at MuxCh1.1 (A4), MuxCh1_5.2 (Pin_2): now also R13.1
- net at MuxCh1.13 (A0), MuxCh1_1.2 (Pin_2): now also R9.1
- net at FX-BTNs1.1 (A4), fx2_btn1.2 (Pin_2): now also R5.1
- net at FX-BTNs1.12 (A3), fx1_btn4.2 (Pin_2): now also R4.1
- net at FX-BTNs1.13 (A0), fx1_btn1.2 (Pin_2): now also R1.1
- net at FX-BTNs1.14 (A1), fx1_btn2.2 (Pin_2): now also R2.1
- net at FX-BTNs1.15 (A2), fx1_btn3.2 (Pin_2): now also R3.1
- net at FX-BTNs1.2 (A6), fx2_btn3.2 (Pin_2): now also R7.1
- net at FX-BTNs1.4 (A7), fx2_btn4.2 (Pin_2): now also R8.1
- net at FX-BTNs1.5 (A5), fx2_btn2.2 (Pin_2): now also R6.1
- new net: R18.1, U5.18 (26_A12_MOSI1)
- new net: R33.2, U5.30 (38_CS1_IN1)
- new net: R32.2, U5.31 (39_MISO1_OUT1A)
- new net: R31.2, U5.32 (40_A16)
- new net: R30.2, U5.33 (41_A17)
- new net: MuxCh1_37.2 (Pin_2), MuxCh5.1 (A4), R64.1
- new net: MuxCh1_38.2 (Pin_2), MuxCh5.5 (A5), R65.1
- new net: MuxCh1_40.2 (Pin_2), MuxCh5.4 (A7), R67.1
- new net: MuxCh1_36.2 (Pin_2), MuxCh5.12 (A3), R63.1
- new net: MuxCh1_39.2 (Pin_2), MuxCh5.2 (A6), R66.1
- new net: MuxCh1_33.2 (Pin_2), MuxCh5.13 (A0), R60.1
- new net: MuxCh1_34.2 (Pin_2), MuxCh5.14 (A1), R61.1
- new net: MuxCh1_35.2 (Pin_2), MuxCh5.15 (A2), R62.1
Other:
- moved on the sheet: MuxCh1, MuxCh1_1, MuxCh1_2, MuxCh1_3, MuxCh1_4, MuxCh1_5, MuxCh1_6, MuxCh1_7, MuxCh1_8

Commit message: mixer-pcb edits
Parts:
- added 3.3V_In1, 3.3V_Test1, 3.3V_Test2: Conn_01x02, Connector_JST:JST_XH_B2B-XH-AM_1x02_P2.50mm_Vertical, symbol Connector_Generic:Conn_01x02
- added C10, C3, C4, C5, C6, C8, C9: 100 nF, Capacitor_THT:CP_Radial_D5.0mm_P2.50mm, symbol Device:C
- added C2, C7: 100 uF, Capacitor_THT:CP_Radial_D10.0mm_P2.50mm, symbol mixer.pcb-rescue:CP-Device
- C1: value CP -> 100 uF
Connections:
- net +3V3: now also 3.3V_In1.1 (Pin_1), 3.3V_Test1.2 (Pin_2), 3.3V_Test2.2 (Pin_2), C10.2, C2.1, C4.2, C5.2, C6.2, C7.2, C8.2, C9.2; no longer C1.2, U5.15 (3V3), U5.46 (3V3)
- net GND: now also C1.2, 3.3V_In1.2 (Pin_2), C10.1, C2.2, C3.1, C4.1, C5.1, C6.1, C7.1, C8.1, C9.1
- new net: 3.3V_Test1.1 (Pin_1), C3.2, U5.15 (3V3)
- new net: 3.3V_Test2.1 (Pin_1), U5.46 (3V3)
Other:
- note added: "Zuleitung"
- moved on the sheet: FX-BTNs1, fxEncBtns1
