File: Controller_Mixer/pcb/controller_mixer_pcb_v0.2/mixer.pcb.sch (KiCad schematic (older format))
At the start: 158 parts, among them U5 Teensy4.1

Commit message: mixer-pcb ready
Parts:
- added C11, C12: 100 nF, Capacitor_THT:CP_Radial_D5.0mm_P2.50mm, symbol Device:C
Connections:
- net +3V3: now also C11.2, C12.2
- net GND: now also C11.1, C12.1
Changed lines of the file:
@@
 $EndComp
 Connection ~ 950  6150
+$Comp
+L Device:C C11
+U 1 1 6040F556
+P 10950 7500
+F 0 "C11" H 11065 7546 50  0001 L CNN
+F 1 "100 nF" H 11065 7455 50  0000 L CNN
+F 2 "Capacitor_THT:CP_Radial_D5.0mm_P2.50mm" H 10988 7350 50  0001 C CNN
+F 3 "~" H 10950 7500 50  0001 C CNN
+	1    10950 7500
+	-1   0    0    1
+$EndComp
+$Comp
+L power:GND #PWR0315
+U 1 1 6040F55C
+P 10950 7650
+F 0 "#PWR0315" H 10950 7400 50  0001 C CNN
+F 1 "GND" V 10955 7522 50  0000 R CNN
+F 2 "" H 10950 7650 50  0001 C CNN
+F 3 "" H 10950 7650 50  0001 C CNN
+	1    10950 7650
+	0    1    -1   0
+$EndComp
+Connection ~ 10950 7350
+$Comp
+L Device:C C12
+U 1 1 60489670
+P 14050 7550
+F 0 "C12" H 14165 7596 50  0001 L CNN
+F 1 "100 nF" H 14165 7505 50  0000 L CNN
+F 2 "Capacitor_THT:CP_Radial_D5.0mm_P2.50mm" H 14088 7400 50  0001 C CNN
+F 3 "~" H 14050 7550 50  0001 C CNN
+	1    14050 7550
+	-1   0    0    1
+$EndComp
+$Comp
+L power:GND #PWR0316
+U 1 1 60489676
+P 14050 7700
+F 0 "#PWR0316" H 14050 7450 50  0001 C CNN
+F 1 "GND" V 14055 7572 50  0000 R CNN
+F 2 "" H 14050 7700 50  0001 C CNN
+F 3 "" H 14050 7700 50  0001 C CNN
+	1    14050 7700
+	0    1    -1   0
+$EndComp
+Connection ~ 14050 7400
 $EndSCHEMATC

Commit message: corrections
Parts:
- 3.3V_In1, 3.3V_Test1, 3.3V_Test2, fx1_btn1, fx1_btn2, fx1_btn3, fx1_btn4, fx2_btn1, fx2_btn2, fx2_btn3, fx2_btn4, pfl_btn_1, pfl_btn_2, pfl_btn_3, pfl_btn_4, pfl_btn_master1, pfl_led_1, pfl_led_2, pfl_led_3, pfl_led_4, pfl_led_master1: symbol Connector_Generic:Conn_01x02 -> mixer.pcb-rescue:Conn_01x02-Connector_Generic
- C10, C11, C12, C3, C4, C5, C6, C8, C9: symbol Device:C -> mixer.pcb-rescue:C-Device
- FX-BTNs1, MuxCh1, MuxCh2, MuxCh3, MuxCh4, MuxCh5, fxEncBtns1: symbol 74xx:74HC4051 -> mixer.pcb-rescue:74HC4051-74xx
- MuxCh1_1, MuxCh1_10, MuxCh1_11, MuxCh1_12, MuxCh1_13, MuxCh1_14, MuxCh1_15, MuxCh1_16, MuxCh1_17, MuxCh1_18, MuxCh1_19, MuxCh1_2, MuxCh1_20, MuxCh1_21, MuxCh1_22, MuxCh1_23, MuxCh1_24, MuxCh1_25, MuxCh1_26, MuxCh1_27, MuxCh1_28, MuxCh1_29, MuxCh1_3, MuxCh1_30, MuxCh1_31, MuxCh1_32, MuxCh1_33, MuxCh1_34, MuxCh1_35, MuxCh1_36, MuxCh1_37, MuxCh1_38, MuxCh1_39, MuxCh1_4, MuxCh1_40, MuxCh1_5, MuxCh1_6, MuxCh1_7, MuxCh1_8, MuxCh1_9, NeoPixel1, spare(28)1, spare(29)1: symbol Connector_Generic:Conn_01x03 -> mixer.pcb-rescue:Conn_01x03-Connector_Generic
- display_1, display_2: symbol Connector_Generic:Conn_01x04 -> mixer.pcb-rescue:Conn_01x04-Connector_Generic
- fx1_enc1, fx1_enc2, fx1_enc3, fx2_enc1, fx2_enc2, fx2_enc3: symbol Connector_Generic:Conn_01x05 -> mixer.pcb-rescue:Conn_01x05-Connector_Generic
Connections:
- net +3V3: now also NeoPixel1.1 (Pin_1), fx1_enc1.1 (Pin_1), fx1_enc2.1 (Pin_1), fx1_enc3.1 (Pin_1), fx2_enc1.1 (Pin_1), fx2_enc2.1 (Pin_1), fx2_enc3.1 (Pin_1), pfl_btn_1.1 (Pin_1), pfl_btn_2.1 (Pin_1), pfl_btn_3.1 (Pin_1), pfl_btn_4.1 (Pin_1), pfl_btn_master1.1 (Pin_1), spare(28)1.1 (Pin_1), spare(29)1.1 (Pin_1); no longer NeoPixel1.3 (Pin_3), fx1_enc1.2 (Pin_2), fx1_enc2.2 (Pin_2), fx1_enc3.2 (Pin_2), fx2_enc1.2 (Pin_2), fx2_enc2.2 (Pin_2), fx2_enc3.2 (Pin_2), pfl_btn_1.2 (Pin_2), pfl_btn_2.2 (Pin_2), pfl_btn_3.2 (Pin_2), pfl_btn_4.2 (Pin_2), pfl_btn_master1.2 (Pin_2), pfl_led_1.2 (Pin_2), pfl_led_2.2 (Pin_2), pfl_led_3.2 (Pin_2), pfl_led_4.2 (Pin_2), pfl_led_master1.2 (Pin_2), spare(28)1.3 (Pin_3), spare(29)1.3 (Pin_3)
- net GND: now also NeoPixel1.3 (Pin_3), fx1_enc1.2 (Pin_2), fx1_enc2.2 (Pin_2), fx1_enc3.2 (Pin_2), fx2_enc1.2 (Pin_2), fx2_enc2.2 (Pin_2), fx2_enc3.2 (Pin_2), pfl_led_1.2 (Pin_2), pfl_led_2.2 (Pin_2), pfl_led_3.2 (Pin_2), pfl_led_4.2 (Pin_2), pfl_led_master1.2 (Pin_2), spare(28)1.3 (Pin_3), spare(29)1.3 (Pin_3); no longer NeoPixel1.1 (Pin_1), fx1_enc1.1 (Pin_1), fx1_enc2.1 (Pin_1), fx1_enc3.1 (Pin_1), fx2_enc1.1 (Pin_1), fx2_enc2.1 (Pin_1), fx2_enc3.1 (Pin_1), spare(28)1.2 (Pin_2), spare(29)1.2 (Pin_2)
- net pfl_btn_ch1: now also pfl_btn_1.2 (Pin_2); no longer pfl_btn_1.1 (Pin_1)
- net pfl_btn_ch2: now also pfl_btn_2.2 (Pin_2); no longer pfl_btn_2.1 (Pin_1)
- net pfl_btn_ch3: now also pfl_btn_3.2 (Pin_2); no longer pfl_btn_3.1 (Pin_1)
- net pfl_btn_ch4: now also pfl_btn_4.2 (Pin_2); no longer pfl_btn_4.1 (Pin_1)
- net pfl_btn_master: now also pfl_btn_master1.2 (Pin_2); no longer pfl_btn_master1.1 (Pin_1)
- net pin28: now also spare(28)1.2 (Pin_2); no longer spare(28)1.1 (Pin_1)
- net pin29: now also spare(29)1.2 (Pin_2); no longer spare(29)1.1 (Pin_1)
