File: Controller_Mixer/pcb/controller_mixer_pcb_v0.2/mixer.pcb.kicad_pcb (KiCad board)
At the start: 4 copper layers, 146 parts, among them U5 Teensy4.1

Commit message: mixer-pcb edits
Parts:
- added 3.3V_In1: Conn_01x02, Connector_JST:JST_XH_B2B-XH-AM_1x02_P2.50mm_Vertical, F.Cu at (160.0, 188.0)
- added 3.3V_Test1: Conn_01x02, Connector_JST:JST_XH_B2B-XH-AM_1x02_P2.50mm_Vertical, F.Cu at (147.3, 213.4)
- added 3.3V_Test2: Conn_01x02, Connector_JST:JST_XH_B2B-XH-AM_1x02_P2.50mm_Vertical, F.Cu at (48.6, 176.5)
- added C10: 100 nF, Capacitor_THT:CP_Radial_D5.0mm_P2.50mm, F.Cu at (166.4, 114.3)
- added C2: 100 uF, Capacitor_THT:CP_Radial_D10.0mm_P2.50mm, F.Cu at (148.6, 179.1)
- added C3: 100 nF, Capacitor_THT:CP_Radial_D5.0mm_P2.50mm, F.Cu at (152.4, 222.2)
- added C4: 100 nF, Capacitor_THT:CP_Radial_D5.0mm_P2.50mm, F.Cu at (26.7, 115.6)
- added C5: 100 nF, Capacitor_THT:CP_Radial_D5.0mm_P2.50mm, F.Cu at (48.5, 167.6)
- added C6: 100 nF, Capacitor_THT:CP_Radial_D5.0mm_P2.50mm, F.Cu at (54.6, 123.2)
- added C7: 100 uF, Capacitor_THT:CP_Radial_D10.0mm_P2.50mm, F.Cu at (27.9, 176.5)
- added C8: 100 nF, Capacitor_THT:CP_Radial_D5.0mm_P2.50mm, F.Cu at (96.5, 115.6)
- added C9: 100 nF, Capacitor_THT:CP_Radial_D5.0mm_P2.50mm, F.Cu at (125.7, 123.2)
- added REF**: MountingHole_2.5mm, MountingHole:MountingHole_2.5mm, F.Cu at (154.9, 68.6)
- added REF**: MountingHole_2.5mm, MountingHole:MountingHole_2.5mm, F.Cu at (16.5, 114.3)
- added REF**: MountingHole_2.5mm, MountingHole:MountingHole_2.5mm, F.Cu at (16.5, 166.4)
- added REF**: MountingHole_2.5mm, MountingHole:MountingHole_2.5mm, F.Cu at (16.5, 218.4)
- added REF**: MountingHole_2.5mm, MountingHole:MountingHole_2.5mm, F.Cu at (148.6, 279.4)
- added REF**: MountingHole_2.5mm, MountingHole:MountingHole_2.5mm, F.Cu at (16.5, 279.4)
- added REF**: MountingHole_2.5mm, MountingHole:MountingHole_2.5mm, F.Cu at (58.4, 279.4)
- added REF**: MountingHole_2.5mm, MountingHole:MountingHole_2.5mm, F.Cu at (102.9, 279.4)
- added REF**: MountingHole_2.5mm, MountingHole:MountingHole_2.5mm, F.Cu at (193.0, 279.4)
- added REF**: MountingHole_2.5mm, MountingHole:MountingHole_2.5mm, F.Cu at (191.8, 219.7)
- added REF**: MountingHole_2.5mm, MountingHole:MountingHole_2.5mm, F.Cu at (191.8, 168.9)
- added REF**: MountingHole_2.5mm, MountingHole:MountingHole_2.5mm, F.Cu at (49.5, 68.6)
- added REF**: MountingHole_2.5mm, MountingHole:MountingHole_2.5mm, F.Cu at (191.8, 118.1)
- added REF**: MountingHole_2.5mm, MountingHole:MountingHole_2.5mm, F.Cu at (191.8, 66.0)
- added REF**: MountingHole_2.5mm, MountingHole:MountingHole_2.5mm, F.Cu at (191.8, 17.8)
- added REF**: MountingHole_2.5mm, MountingHole:MountingHole_2.5mm, F.Cu at (135.9, 17.8)
- added REF**: MountingHole_2.5mm, MountingHole:MountingHole_2.5mm, F.Cu at (64.8, 17.8)
- added REF**: MountingHole_2.5mm, MountingHole:MountingHole_2.5mm, F.Cu at (16.5, 16.5)
- added REF**: MountingHole_2.5mm, MountingHole:MountingHole_2.5mm, F.Cu at (83.8, 68.6)
- added REF**: MountingHole_2.5mm, MountingHole:MountingHole_2.5mm, F.Cu at (120.7, 68.6)
- added REF**: MountingHole_2.5mm, MountingHole:MountingHole_2.5mm, F.Cu at (147.3, 204.5)
- added REF**: MountingHole_2.5mm, MountingHole:MountingHole_2.5mm, F.Cu at (90.2, 240.0)
- added REF**: MountingHole_2.5mm, MountingHole:MountingHole_2.5mm, F.Cu at (58.4, 210.8)
- added REF**: MountingHole_2.5mm, MountingHole:MountingHole_2.5mm, F.Cu at (99.1, 124.5)
- added REF**: MountingHole_2.5mm, MountingHole:MountingHole_2.5mm, F.Cu at (16.5, 62.2)
- C1: value CP -> 100 uF
- moved C1 3.81 mm to (27.9, 189.2)
Connections:
- C1 pad 2: +3V3 -> GND
- U5 pad 15: +3V3 -> Net-(3.3V_Test1-Pad1)
- U5 pad 46: +3V3 -> Net-(3.3V_Test2-Pad1)
Routing:
- net Net-(3.3V_Test1-Pad1): track 0.00 -> 66.1 mm, vias 0 -> 1
- net Net-(3.3V_Test2-Pad1): track 0.00 -> 54.7 mm, vias 0 -> 2
- net s0: track 519.4 -> 502.8 mm
- net s2: track 470.7 -> 455.7 mm
- net s1: track 494.2 -> 479.4 mm
- net pin28: track 120.7 -> 112.5 mm, vias 3 -> 1
- net pin29: track 106.7 -> 101.5 mm, vias 3 -> 1
- net display_scl2: track 99.1 -> 94.4 mm, vias 3 -> 1
- net display_sda2: track 96.6 -> 92.7 mm, vias 3 -> 1
- net +3V3: track 12.8 -> 8.97 mm
- net Net-(fx2_enc2-Pad3): track 88.9 -> 87.4 mm, vias 4 -> 3
- net rEnc5_clk: track 124.5 -> 123.0 mm, vias 2 -> 1
- net rEnc4_DT: track 116.9 -> 115.4 mm, vias 2 -> 1
- net rEnc5_DT: track 129.6 -> 128.1 mm, vias 2 -> 1
- net rEnc2_clk: track 104.2 -> 103.5 mm, vias 3 -> 1
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
Commit message: corrections
Parts:
- removed the REF** at (16.5, 114.3)
- removed the REF** at (191.8, 219.7)
- removed the REF** at (191.8, 168.9)
- removed the REF** at (191.8, 118.1)
- removed the REF** at (191.8, 66.0)
- removed the REF** at (191.8, 17.8)
- removed the REF** at (135.9, 17.8)
- removed the REF** at (64.8, 17.8)
- removed the REF** at (147.3, 204.5)
- removed the REF** at (58.4, 210.8)
- removed the REF** at (99.1, 124.5)
- removed the REF** at (16.5, 62.2)
- added REF**: MountingHole_2.5mm, MountingHole:MountingHole_2.5mm, F.Cu at (16.5, 118.1)
- added REF**: MountingHole_2.5mm, MountingHole:MountingHole_2.5mm, F.Cu at (191.8, 218.4)
- added REF**: MountingHole_2.5mm, MountingHole:MountingHole_2.5mm, F.Cu at (193.0, 166.4)
- added REF**: MountingHole_2.5mm, MountingHole:MountingHole_2.5mm, F.Cu at (193.0, 118.1)
- added REF**: MountingHole_2.5mm, MountingHole:MountingHole_2.5mm, F.Cu at (193.0, 68.6)
- added REF**: MountingHole_2.5mm, MountingHole:MountingHole_2.5mm, F.Cu at (193.0, 16.5)
- added REF**: MountingHole_2.5mm, MountingHole:MountingHole_2.5mm, F.Cu at (135.9, 16.5)
- added REF**: MountingHole_2.5mm, MountingHole:MountingHole_2.5mm, F.Cu at (64.8, 16.5)
- added REF**: MountingHole_2.5mm, MountingHole:MountingHole_2.5mm, F.Cu at (146.1, 205.7)
- added REF**: MountingHole_2.5mm, MountingHole:MountingHole_2.5mm, F.Cu at (61.0, 205.7)
- added REF**: MountingHole_2.5mm, MountingHole:MountingHole_2.5mm, F.Cu at (97.8, 118.1)
- added REF**: MountingHole_2.5mm, MountingHole:MountingHole_2.5mm, F.Cu at (16.5, 68.6)
- moved 3.3V_Test2 20.8 mm to (27.9, 179.1)
- moved C6 18.2 mm to (72.4, 119.4), turned to 90 degrees
- moved C9 18.2 mm to (143.5, 119.4), turned to 90 degrees
- moved C10 17.1 mm to (177.8, 101.6), turned to 90 degrees
- moved C8 17.1 mm to (108.0, 102.9), turned to 90 degrees
- moved C4 16.3 mm to (36.8, 102.9), turned to 90 degrees
- moved C5 13.3 mm to (36.8, 174.0), turned to 180 degrees
- moved R41 12.7 mm to (102.9, 158.8)
- moved C7 10.2 mm to (27.9, 166.4), turned to 270 degrees
- moved R40 7.62 mm to (102.9, 168.9)
- moved 3.3V_Test1 6.35 mm to (147.3, 219.7)
- moved R39 6.35 mm to (102.9, 172.7)
- moved R42 5.08 mm to (102.9, 180.3)
- moved C3 4.58 mm to (156.2, 219.7), turned to 180 degrees
- moved R43 3.81 mm to (102.9, 176.5)
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Routing:
- net Net-(3.3V_Test2-Pad1): track 54.7 -> 72.9 mm
- net pfl_btn_ch3: track 98.1 -> 81.5 mm, vias 3 -> 2
- net Net-(FX-BTNs1-Pad12): track 68.4 -> 59.5 mm, vias 3 -> 2
- net pin29: track 101.5 -> 93.3 mm
- net Net-(3.3V_Test1-Pad1): track 66.1 -> 60.3 mm
- net pin28: track 112.5 -> 107.3 mm
- net display_sda2: track 92.7 -> 87.6 mm
- net pfl_btn_ch2: track 170.0 -> 164.9 mm
- net display_scl2: track 94.4 -> 89.3 mm
- net pfl_btn_ch1: track 190.5 -> 194.3 mm
- net pfl_btn_ch4: track 105.4 -> 107.9 mm, vias 2 -> 3
- net Net-(MuxCh1-Pad2): track 34.1 -> 32.0 mm, vias 0 -> 2
- net Net-(fx1_enc3-Pad3): track 127.3 -> 125.9 mm
- net rEnc0_clk: track 58.5 -> 57.0 mm
- net mux_encBtn_fx: track 85.6 -> 84.1 mm
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