File: Controller_Mixer/pcb/controller_mixer_pcb_v0.2/mixer.pcb.kicad_pcb (KiCad board)
At the start: 4 copper layers, 184.2 x 270.5 mm, 185 parts, among them U5 Teensy4.1

Commit message: pcb v0.2 - this went to jlcpcb and hopefully it works this time.
Parts:
- moved NeoPixel1 11.4 mm to (27.9, 191.8)
- moved C1 10.2 mm to (26.7, 199.4), turned to 270 degrees
- renumbered 3.3V_In1 to 3.3V_In, MuxCh1_9 to MuxCh2_1, MuxCh1_10 to MuxCh2_2, MuxCh1_11 to MuxCh2_3, MuxCh1_12 to MuxCh2_4, MuxCh1_13 to MuxCh2_5, MuxCh1_14 to MuxCh2_6, MuxCh1_15 to MuxCh2_7, MuxCh1_16 to MuxCh2_8, MuxCh1_17 to MuxCh3_1, MuxCh1_18 to MuxCh3_2, MuxCh1_19 to MuxCh3_3, MuxCh1_20 to MuxCh3_4, MuxCh1_21 to MuxCh3_5, MuxCh1_22 to MuxCh3_6, MuxCh1_23 to MuxCh3_7, MuxCh1_24 to MuxCh3_8, MuxCh1_25 to MuxCh4_1, MuxCh1_26 to MuxCh4_2, MuxCh1_27 to MuxCh4_3, MuxCh1_28 to MuxCh4_4, MuxCh1_29 to MuxCh4_5, MuxCh1_30 to MuxCh4_6, MuxCh1_31 to MuxCh4_7, MuxCh1_32 to MuxCh4_8, MuxCh1_33 to MuxCh5_1, MuxCh1_34 to MuxCh5_2, MuxCh1_35 to MuxCh5_3, MuxCh1_36 to MuxCh5_4, MuxCh1_37 to MuxCh5_5, MuxCh1_38 to MuxCh5_6, MuxCh1_39 to MuxCh5_7, MuxCh1_40 to MuxCh5_8, spare(28)1 to spare28, spare(29)1 to spare29, VU_Matrix1 to vu_matrix
Routing:
- net +3V3: track 8.97 -> 0.00 mm
- net neopixel: track 80.0 -> 88.6 mm
Other:
- board text added: "+"
- board text added: "M"
