File: hardware/moc/btn-matrix_pcb/btn-matrix.sch (KiCad schematic (older format))
At the start: 97 parts, among them J2 Conn_02x12_Odd_Even, U0 WS2811, U1 WS2811, U10 WS2811, U11 WS2811, U12 WS2811, U13 WS2811, U14 WS2811, U15 WS2811, U2 WS2811, U3 WS2811, U4 WS2811, U5 WS2811, U6 WS2811, U7 WS2811, U8 WS2811, U9 WS2811

Commit message: CC BY-NC-SA 4.0 license for hardware ready
Parts:
- added H1, H2, H3, H4, H5: MountingHole_Pad, MountingHole:MountingHole_2.7mm_Pad_Via, symbol btn-matrix-rescue:MountingHole_Pad-Mechanical
- C0, C1, C10, C11, C12, C13, C14, C15, C2, C3, C4, C5, C6, C7, C8, C9: symbol Device:C -> btn-matrix-rescue:C-Device
- J2: symbol Connector_Generic:Conn_02x12_Odd_Even -> btn-matrix-rescue:Conn_02x12_Odd_Even-Connector_Generic
- R0.1, R0.2, R0.3, R1.1, R1.2, R1.3, R10.1, R10.2, R10.3, R11.1, R11.2, R11.3, R12.1, R12.2, R12.3, R13.1, R13.2, R13.3, R14.1, R14.2, R14.3, R15.1, R15.2, R15.3, R2.1, R2.2, R2.3, R3.1, R3.2, R3.3, R4.1, R4.2, R4.3, R5.1, R5.2, R5.3, R6.1, R6.2, R6.3, R7.1, R7.2, R7.3, R8.1, R8.2, R8.3, R9.1, R9.2, R9.3: symbol Device:R -> btn-matrix-rescue:R-Device
- S0, S1, S10, S11, S12, S13, S14, S15, S2, S3, S4, S5, S6, S7, S8, S9: symbol SamacSys_Parts:228CMVARGBFR -> btn-matrix-rescue:228CMVARGBFR-SamacSys_Parts
- U0, U1, U10, U11, U12, U13, U14, U15, U2, U3, U4, U5, U6, U7, U8, U9: symbol Driver_LED:WS2811 -> btn-matrix-rescue:WS2811-Driver_LED
Connections:
- wire segments 253 -> 262
