File: a3motion/mocHardware/Mainboard-pcb/controller_motion_pcb.kicad_pcb (KiCad board)
At the start: 2 copper layers, 30 x 156 mm, 42 parts, among them J1 SPI_Female, J2 SPI_Male, J3 Conn_01x06_Female, J4 UPDI_Interface, J5 Programm_Jumper, SW1 Rotary_Encoder_Switch, U1 TPIC6C595-SOIC, U2 TPIC6C595-SOIC, U3 ATtiny1626

Commit message: cleaned libs and finished main und rpi pcb
Parts:
- added REF**: MountingHole_3.2mm_M3, MountingHole:MountingHole_3.2mm_M3, F.Cu at (144.1, 20.4)
- added REF**: MountingHole_3.2mm_M3, MountingHole:MountingHole_3.2mm_M3, F.Cu at (144.1, 174.5)
- S1, S2, S3, S4: footprint MOUSERfootprintANDsymbol:228CMVARGBFR -> 3dAudioFoot:228CMVARGBFR_SMD
- SW1: footprint MOUSERfootprintANDsymbol:PEC11R4230KS0024 -> 3dAudioFoot:PEC11R4230KS0024
- U1, U2: value TPIC6C595-SOIC -> TPIC6C595
- U3: footprint .Ambisonic:attiny1626 -> 3dAudioFoot:attiny1626
- moved C2 4.97 mm to (131.8, 40.8)
- moved R18 4.97 mm to (131.8, 44.3)
- moved C1 4.97 mm to (131.8, 36.3)
- moved R17 4.97 mm to (131.8, 32.8)
Routing:
- net VCC_w: track 121.1 -> 130.2 mm, vias 3 -> 5
- net ENCB: track 99.5 -> 94.2 mm
- net Net-(R18-Pad2): track 4.63 -> 9.54 mm
- net ENCA: track 89.7 -> 84.8 mm
- net GND: track 174.3 -> 178.4 mm, vias 5 -> 7
- net UPDI_w: track 53.4 -> 56.3 mm
- net SDA: track 76.5 -> 78.8 mm
- net SCL: track 76.8 -> 78.0 mm
Other:
- board size 30 x 156 mm -> 30 x 161.5 mm
