File: a3motion/mocHardware/RPIconnector/rpiconnector/rpiconnector.kicad_sch (KiCad schematic)
At the start: 9 parts, among them J1 Conn_01x05_Male, J2 Conn_02x05_Odd_Even, Q1 BSS138, Q2 BSS138, U1 USB-C

Commit message: cleaned libs and finished main und rpi pcb
Parts:
- removed U1: USB-C, .Ambisonic:USB-C, symbol .Ambisonic:USB-C
- added U1: USB-C, 3dAudioFoot:USB-C, symbol 3dAudioSym:USB-C
Connections:
- net 5v: now also U1.2 (VBUS), U1.5 (VBUS)
- net GND: now also U1.1 (GND), U1.6 (GND)
Changed lines of the file:
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@@
     (pin "2")
   )
-  (symbol (lib_id ".Ambisonic:USB-C") (at 45.72 102.87 0) (unit 1)
+  (symbol (lib_id "3dAudioSym:USB-C") (at 45.72 102.87 0) (unit 1)
     (in_bom yes) (on_board yes) (fields_autoplaced)
     (property "Reference" "U1" (id 0) (at 41.275 93.8743 0))
     (property "Value" "USB-C" (id 1) (at 41.275 96.6494 0))
-    (property "Footprint" ".Ambisonic:USB-C" (id 2) (at 45.72 102.87 0)
+    (property "Footprint" "3dAudioFoot:USB-C" (id 2) (at 45.72 102.87 0)
       (effects (font (size 1.27 1.27)) hide)
     )
@@
       (reference "R4") (unit 1) (value "10k") (footprint "Resistor_SMD:R_1206_3216Metric_Pad1.30x1.75mm_HandSolder")
     )
-    (path "/3cbb223f-d0e4-484b-8711-77e5036b15b5"
-      (reference "U1") (unit 1) (value "USB-C") (footprint ".Ambisonic:USB-C")
+    (path "/39ac7e3c-47f1-43e5-b70d-8dfebc468916"
+      (reference "U1") (unit 1) (value "USB-C") (footprint "3dAudioFoot:USB-C")
     )
   )
